File: kicad/led_board/led_board.kicad_pcb (KiCad board)
At the start: 2 copper layers, 140 x 30 mm, 21 parts, among them J1 MAIN_BOARD

Commit message: kicad: add copyright and license to kicad documents
Parts:
- added G***: LOGO, led_board:oshw_logo, F.Cu at (51.0, 50.8)
Other:
- board text added: "PiModem - LED Board"
- board text added: "Rev 1.0"
