File: kicad/piHAT/pimodem.kicad_pcb (KiCad board)
At the start: 4 copper layers, 65 x 56.5 mm, 40 parts, among them J1 PWR_HEADER, J2 PI_HEADER, J3 SERIAL, J4 AUDIO_HEADER, J5 LED_PANEL, J7 GAIN, Q1 DMG2305UX, Q2 BC857BS, Q3 DMG3414U, U1 LTC2951-2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

Commit message: kicad: add copyright and license to kicad documents
Parts:
- added G***: LOGO, piHAT:oshw_logo, B.Cu at (74.9, 70.1)
